Commit message: Complete ros2_control integration: gazebo, controllers, relay, TF, scan

File: ros2_ws/src/learning_robot/urdf/mobile_robot.urdf.xacro (robot description, xacro)
@@ -119,5 +119,5 @@
         <axis xyz="0 1 0" />
     </joint>
-    <!-- ============ 万向轮 ============ -->
+    <!-- ============ 后万向轮 ============ -->
     <link name="caster_link">
         <visual>
@@ -148,28 +148,33 @@
         <origin xyz="-0.15 0 ${-base_height/2 - 0.03}" rpy="0 0 0" />
     </joint>
-    <!-- ============ Gazebo 差速驱动插件 ============ -->
-    <gazebo>
-        <plugin filename="gz-sim-diff-drive-system"
-            name="gz::sim::systems::DiffDrive">
-            <left_joint>base_to_left_wheel</left_joint>
-            <right_joint>base_to_right_wheel</right_joint>
-            <wheel_separation>0.34</wheel_separation>
-            <wheel_radius>0.05</wheel_radius>
-            <max_linear_acceleration>1.0</max_linear_acceleration>
-            <min_linear_acceleration>-1.0</min_linear_acceleration>
-            <max_angular_acceleration>2.0</max_angular_acceleration>
-            <min_angular_acceleration>-2.0</min_angular_acceleration>
-            <max_linear_velocity>0.5</max_linear_velocity>
-            <min_linear_velocity>-0.5</min_linear_velocity>
-            <max_angular_velocity>1.0</max_angular_velocity>
-            <min_angular_velocity>-1.0</min_angular_velocity>
-            <topic>cmd_vel</topic>
-            <odom_topic>odom</odom_topic>
-            <tf_topic>tf</tf_topic>
-            <frame_id>odom</frame_id>
-            <child_frame_id>base_link</child_frame_id>
-            <odom_publish_frequency>50</odom_publish_frequency>
-        </plugin>
-    </gazebo>
+    <!-- ============ 前万向轮 ============ -->
+    <link name="front_caster_link">
+        <visual>
+            <geometry>
+                <sphere radius="${caster_radius}" />
+            </geometry>
+            <material name="black" />
+        </visual>
+        <collision>
+            <geometry>
+                <sphere radius="${caster_radius}" />
+            </geometry>
+        </collision>
+        <inertial>
+            <origin xyz="0 0 0" rpy="0 0 0" />
+            <mass value="${caster_mass}" />
+            <inertia
+                ixx="${2*caster_mass*caster_radius*caster_radius/5}"
+                ixy="0.0" ixz="0.0"
+                iyy="${2*caster_mass*caster_radius*caster_radius/5}"
+                iyz="0.0"
+                izz="${2*caster_mass*caster_radius*caster_radius/5}" />
+        </inertial>
+    </link>
+    <joint name="base_to_front_caster" type="fixed">
+        <parent link="base_link" />
+        <child link="front_caster_link" />
+        <origin xyz="0.15 0 ${-base_height/2 - 0.03}" rpy="0 0 0" />
+    </joint>
     <!-- 万向轮摩擦系数改为 0，让它能在平面上滑动 -->
     <gazebo reference="caster_link">
@@ -177,4 +182,8 @@
         <mu2>0.0</mu2>
     </gazebo>
+    <gazebo reference="front_caster_link">
+        <mu1>0.0</mu1>
+        <mu2>0.0</mu2>
+    </gazebo>
     <!-- 轮子摩擦系数调高，保证抓地力 -->
     <gazebo reference="left_wheel_link">
@@ -186,3 +195,75 @@
         <mu2>1.0</mu2>
     </gazebo>
+    <!-- ============ ros2_control 硬件接口声明 ============ -->
+    <ros2_control name="GazeboSystem" type="system">
+        <hardware>
+            <plugin>gz_ros2_control/GazeboSimSystem</plugin>
+        </hardware>
+        <joint name="base_to_left_wheel">
+            <command_interface name="velocity">
+                <param name="min">-10</param>
+                <param name="max">10</param>
+            </command_interface>
+            <state_interface name="velocity" />
+            <state_interface name="position" />
+        </joint>
+        <joint name="base_to_right_wheel">
+            <command_interface name="velocity">
+                <param name="min">-10</param>
+                <param name="max">10</param>
+            </command_interface>
+            <state_interface name="velocity" />
+            <state_interface name="position" />
+        </joint>
+    </ros2_control>
+    <!-- ============ gz_ros2_control Gazebo 插件 ============ -->
+    <gazebo>
+        <plugin filename="libgz_ros2_control-system.so"
+            name="gz_ros2_control::GazeboSimROS2ControlPlugin">
+            <parameters>$(find learning_robot)/config/controllers.yaml</parameters>
+        </plugin>
+    </gazebo>
+    <!-- ============ 激光雷达 ============ -->
+    <xacro:property name="lidar_radius" value="0.03" />
+    <xacro:property name="lidar_height" value="0.04" />
+    <xacro:property name="lidar_mass" value="0.1" />
+    <xacro:cylinder_link
+        name="lidar_link"
+        radius="${lidar_radius}" length="${lidar_height}"
+        mass="${lidar_mass}" color="black" />
+    <joint name="base_to_lidar" type="fixed">
+        <parent link="base_link" />
+        <child link="lidar_link" />
+        <origin xyz="0 0 ${base_height/2 + lidar_height/2}" rpy="0 0 0" />
+    </joint>
+    <!-- ============ Gazebo 激光雷达传感器插件 ============ -->
+    <gazebo reference="lidar_link">
+        <sensor name="lidar" type="gpu_lidar">
+            <topic>scan</topic>
+            <gz_frame_id>lidar_link</gz_frame_id>
+            <update_rate>10</update_rate>
+            <always_on>true</always_on>
+            <visualize>true</visualize>
+            <lidar>
+                <scan>
+                    <horizontal>
+                        <samples>360</samples>
+                        <resolution>1</resolution>
+                        <min_angle>-3.14159</min_angle>
+                        <max_angle>3.14159</max_angle>
+                    </horizontal>
+                </scan>
+                <range>
+                    <min>0.1</min>
+                    <max>10.0</max>
+                    <resolution>0.01</resolution>
+                </range>
+                <noise>
+                    <type>gaussian</type>
+                    <mean>0.0</mean>
+                    <stddev>0.01</stddev>
+                </noise>
+            </lidar>
+        </sensor>
+    </gazebo>
 </robot>
